Commit message: Update BRTIRUS2110A_robot.urdf

File: BRTIRUS2110A_description/urdf/BRTIRUS2110A_robot.urdf (robot description, URDF)
Before this commit: robot BRTIRUS2110A, 7 links, 6 joints
Joints:
- joint j1: axis 0 1 0 -> 0 0 1
- joint j4: axis 0 0 1 -> 1 0 0
- joint j5: axis 1 0 0 -> 0 0 1; origin xyz=0 0 0.198 rpy=1.57079632679 0 0 -> xyz=0.829 0 0 rpy=1.57079632679 0 0
- joint j6: axis 0 0 1 -> 1 0 0; origin xyz=0 0.107 0 rpy=1.57079632679 0 0 -> xyz=0.097 0 0 rpy=0 0 0
